File: KiCad/Nooky.kicad_sch (KiCad schematic)
At the start: 8 parts, among them J1 USB A Input, J2 VIN (5 - 7VDC), J3 VADJ (2.85VDC), J4 VADJ (2.85VDC), U1 LM317 / LM350 / LM338 Regulat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

Commit message: Review
Parts:
- added F1: 1A Max, symbol Device:Fuse
- added SW1: Power, symbol Switch:SW_SPST
Connections:
- net at J1.1 (VBUS), J2.1: now also F1.1; no longer U1.1 (VIN)
- new net: F1.2, SW1.1 (A)
- new net: SW1.2 (B), U1.1 (VIN)
Other:
- moved on the sheet: D1, J1, J2, J3, J4, R1, R2, U1

Commit message: Update
Parts:
- J3, J4: value VADJ (2.85VDC) -> VADJ (3.25VDC Unloaded)
- R1: value 1R -> 1R 1W
- U1: value LM317 / LM350 / LM338 Regulator Module (VADJ 2.85VDC) -> LM317/LM350/LM338 Regulator Module (VADJ 3.25VDC)
Other:
- note added: "2.90VDC Loaded"
- moved on the sheet: R1
Changed lines of the file:
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@@
 		(title "Nooky")
 		(date "2026-05-05")
-		(rev "1")
+		(rev "1.1")
 		(company "Illusion Interactive")
 	)
@@
 	(text "Optional"
 		(exclude_from_sim no)
-		(at 147.066 90.424 0)
+		(at 147.32 96.012 0)
+		(effects
+			(font
+				(size 1.27 1.27)
+			)
+		)
+	)
+	(text "2.90VDC Loaded"
+		(exclude_from_sim no)
+		(at 193.548 102.362 0)
 		(effects
 			(font
@@
 	)
 	(junction
-		(at 153.67 93.98)
-		(diameter 0)
-		(color 0 0 0 0)
-	)
-	(junction
 		(at 140.97 93.98)
 		(diameter 0)
@@
 	)
 	(junction
+		(at 153.67 93.98)
+		(diameter 0)
+		(color 0 0 0 0)
+	)
+	(junction
 		(at 96.52 101.6)
 		(diameter 0)
@@
 	(wire
 		(pts
-			(xy 140.97 93.98) (xy 140.97 87.63)
+			(xy 140.97 93.98) (xy 140.97 91.44)
+		)
+		(stroke
+			(width 0)
+			(type solid)
+		)
+	)
+	(wire
+		(pts
+			(xy 170.18 95.25) (xy 170.18 93.98)
+		)
+		(stroke
+			(width 0)
+			(type default)
+		)
+	)
+	(wire
+		(pts
+			(xy 100.33 77.47) (xy 92.71 77.47)
 		)
 		(stroke
@@
 	(wire
 		(pts
-			(xy 170.18 95.25) (xy 170.18 93.98)
-		)
-		(stroke
-			(width 0)
-			(type default)
-		)
-	)
-	(wire
-		(pts
-			(xy 100.33 77.47) (xy 92.71 77.47)
+			(xy 140.97 93.98) (xy 140.97 97.79)
+		)
+		(stroke
+			(width 0)
+			(type default)
+		)
+	)
+	(wire
+		(pts
+			(xy 139.7 97.79) (xy 140.97 97.79)
+		)
+		(stroke
+			(width 0)
+			(type default)
+		)
+	)
+	(wire
+		(pts
+			(xy 140.97 91.44) (xy 144.78 91.44)
+		)
+		(stroke
+			(width 0)
+			(type solid)
+		)
+	)
+	(wire
+		(pts
+			(xy 179.07 110.49) (xy 179.07 99.06)
+		)
+		(stroke
+			(width 0)
+			(type default)
+		)
+	)
+	(wire
+		(pts
+			(xy 184.15 93.98) (xy 184.15 105.41)
+		)
+		(stroke
+			(width 0)
+			(type default)
+		)
+	)
+	(wire
+		(pts
+			(xy 96.52 101.6) (xy 121.92 101.6)
+		)
+		(stroke
+			(width 0)
+			(type default)
+		)
+	)
+	(wire
+		(pts
+			(xy 140.97 93.98) (xy 153.67 93.98)
 		)
 		(stroke
@@
 	(wire
 		(pts
-			(xy 140.97 93.98) (xy 140.97 97.79)
-		)
-		(stroke
-			(width 0)
-			(type default)
-		)
-	)
-	(wire
-		(pts
-			(xy 139.7 97.79) (xy 140.97 97.79)
-		)
-		(stroke
-			(width 0)
-			(type default)
-		)
-	)
-	(wire
-		(pts
-			(xy 140.97 87.63) (xy 144.78 87.63)
+			(xy 139.7 101.6) (xy 160.02 101.6)
+		)
+		(stroke
+			(width 0)
+			(type default)
+		)
+	)
+	(wire
+		(pts
+			(xy 96.52 82.55) (xy 92.71 82.55)
 		)
 		(stroke
@@
 	(wire
 		(pts
-			(xy 179.07 110.49) (xy 179.07 99.06)
-		)
-		(stroke
-			(width 0)
-			(type default)
-		)
-	)
-	(wire
-		(pts
-			(xy 184.15 93.98) (xy 184.15 105.41)
-		)
-		(stroke
-			(width 0)
-			(type default)
-		)
-	)
-	(wire
-		(pts
-			(xy 96.52 101.6) (xy 121.92 101.6)
-		)
-		(stroke
-			(width 0)
-			(type default)
-		)
-	)
-	(wire
-		(pts
-			(xy 140.97 93.98) (xy 153.67 93.98)
-		)
-		(stroke
-			(width 0)
-			(type dash)
-		)
-	)
-	(wire
-		(pts
-			(xy 139.7 101.6) (xy 160.02 101.6)
-		)
-		(stroke
-			(width 0)
-			(type default)
-		)
-	)
-	(wire
-		(pts
-			(xy 96.52 82.55) (xy 92.71 82.55)
-		)
-		(stroke
-			(width 0)
-			(type dash)
-		)
-	)
-	(wire
-		(pts
-			(xy 149.86 87.63) (xy 153.67 87.63)
-		)
-		(stroke
-			(width 0)
-			(type dash)
+			(xy 149.86 91.44) (xy 153.67 91.44)
+		)
+		(stroke
+			(width 0)
+			(type solid)
 		)
 	)
@@
 	(wire
 		(pts
-			(xy 153.67 87.63) (xy 153.67 93.98)
-		)
-		(stroke
-			(width 0)
-			(type dash)
+			(xy 153.67 91.44) (xy 153.67 93.98)
+		)
+		(stroke
+			(width 0)
+			(type solid)
 		)
 	)
@@
 	(symbol
 		(lib_id "Device:R_Small_US")
-		(at 147.32 87.63 270)
+		(at 147.32 91.44 270)
 		(unit 1)
 		(body_style 1)
@@
 		(in_pos_files yes)
 		(dnp no)
-		(fields_autoplaced yes)
 		(property "Reference" "R1"
-			(at 147.32 81.28 90)
-			(show_name no)
-			(do_not_autoplace no)
-			(effects
-				(font
-					(size 1.27 1.27)
-				)
-			)
-		)
-		(property "Value" "1R"
-			(at 147.32 83.82 90)
+			(at 147.32 85.852 90)
+			(show_name no)
+			(do_not_autoplace no)
+			(effects
+				(font
+					(size 1.27 1.27)
+				)
+			)
+		)
+		(property "Value" "1R 1W"
+			(at 147.32 88.392 90)
 			(show_name no)
 			(do_not_autoplace no)
@@
 		)
 		(property "Footprint" ""
-			(at 147.32 87.63 0)
+			(at 147.32 91.44 0)
 			(hide yes)
 			(show_name no)
@@
 		)
 		(property "Datasheet" ""
-			(at 147.32 87.63 0)
+			(at 147.32 91.44 0)
 			(hide yes)
 			(show_name no)
@@
 		)
 		(property "Description" "Resistor, small US symbol"
-			(at 147.32 87.63 0)
+			(at 147.32 91.44 0)
 			(hide yes)
 			(show_name no)
@@
 			)
 		)
-		(property "Value" "VADJ (2.85VDC)"
+		(property "Value" "VADJ (3.25VDC Unloaded)"
 			(at 193.04 90.17 0)
 			(show_name no)
@@
 			)
 		)
-		(property "Value" "VADJ (2.85VDC)"
+		(property "Value" "VADJ (3.25VDC Unloaded)"
 			(at 193.294 116.84 0)
 			(show_name no)
@@
 			)
 		)
-		(property "Value" "LM317 / LM350 / LM338 Regulator Module (VADJ 2.85VDC)"
+		(property "Value" "LM317/LM350/LM338 Regulator Module (VADJ 3.25VDC)"
 			(at 130.556 105.918 0)
 			(show_name no)
